File: stereophonic-amp.kicad_pcb (KiCad board)
At the start: 2 copper layers, 58 parts, among them J1 DIN-3, J2 Headphones, Q1 ГТ308В, Q10 П217Б, Q2 МП26, Q3 МП26, Q4 МП38А, Q5 МП41А, Q6 МП41А, Q7 ГТ402В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

Commit message: Route tone control block
Parts:
- moved C7 194.5 mm to (97.8, 87.6), turned to 90 degrees
- moved C4 187.7 mm to (88.9, 110.5), turned to 90 degrees
- moved R7 161.7 mm to (97.8, 97.8), turned to 180 degrees
- moved C8 161.0 mm to (109.2, 97.8)
- moved RV3 159.0 mm to (90.2, 92.7), turned to 90 degrees
- moved C5 155.7 mm to (97.8, 113.0), turned to 90 degrees
- moved RV2 154.2 mm to (90.2, 102.9), turned to 90 degrees
- moved R8 139.5 mm to (110.5, 102.9), turned to 270 degrees
- moved R6 133.2 mm to (102.9, 102.9), turned to 90 degrees
- moved Q2 129.6 mm to (120.7, 97.8), turned to 270 degrees
- moved RV4 126.7 mm to (135.9, 108.0)
- moved R10 16.1 mm to (224.8, 106.7), turned to 270 degrees
- moved C6 15.3 mm to (88.9, 85.1), turned to 270 degrees
- moved C3 11.7 mm to (74.9, 87.6)
- moved R5 9.25 mm to (81.3, 92.7)
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Routing:
- net Net-(C1-Pad2): track 26.9 -> 0.00 mm
- net Net-(Q1-Pad2): track 17.4 -> 0.00 mm
- net Net-(C3-Pad2): track 16.8 -> 0.00 mm
- net Net-(C2-Pad1): track 10.8 -> 0.00 mm

Commit message: Trace first cascades of amplifier
Parts:
- Q10, Q6, Q9: footprint Connector_PinHeader_1.00mm:PinHeader_1x03_P1.00mm_Vertical -> Connector_PinHeader_2.54mm:PinHeader_1x03_P2.54mm_Vertical
- RV4, RV5: footprint Potentiometer_THT:Potentiometer_Piher_PT-15-V15_Vertical -> Potentiometer_THT:Potentiometer_Piher_PT-10-V10_Vertical
- moved R11 209.6 mm to (67.3, 94.0)
- moved R9 203.5 mm to (53.3, 67.3)
- moved Q3 201.4 mm to (87.6, 72.4), turned to 270 degrees
- moved C9 197.6 mm to (87.6, 86.4), turned to 90 degrees
- moved C10 175.5 mm to (90.2, 50.8), turned to 180 degrees
- moved C11 175.0 mm to (109.2, 80.0), turned to 90 degrees
- moved D2 169.0 mm to (53.3, 78.7)
- moved Q6 168.1 mm to (100.3, 97.8), turned to 180 degrees
- moved Q8 166.9 mm to (119.4, 76.2)
- moved R15 158.1 mm to (77.5, 83.8), turned to 180 degrees
- moved Q10 155.9 mm to (143.5, 81.3), turned to 90 degrees
- moved Q9 155.8 mm to (143.5, 73.7), turned to 90 degrees
- moved D1 155.5 mm to (81.3, 102.9)
- moved R12 155.2 mm to (96.5, 72.4), turned to 270 degrees
- moved Q4 154.8 mm to (85.1, 59.7)
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Routing:
- net Net-(D4-Pad2): track 0.00 -> 79.5 mm
- net Net-(C10-Pad1): track 0.00 -> 71.2 mm
- net Net-(Q5-Pad2): track 0.00 -> 66.4 mm
- net Net-(C10-Pad2): track 0.00 -> 53.8 mm
- net Net-(C3-Pad2): track 0.00 -> 51.8 mm
- net Net-(D3-Pad1): track 0.00 -> 38.8 mm
- net Net-(D2-Pad2): track 0.00 -> 38.8 mm
- net Net-(C3-Pad1): track 0.00 -> 37.5 mm
- net Net-(C11-Pad1): track 0.00 -> 33.9 mm
- net Net-(D2-Pad1): track 0.00 -> 30.1 mm
- net Net-(C4-Pad1): track 0.00 -> 28.3 mm
- net Net-(C1-Pad2): track 0.00 -> 24.5 mm
- net Net-(D1-Pad1): track 0.00 -> 22.7 mm
- net Net-(C11-Pad2): track 0.00 -> 22.7 mm
- net Net-(C8-Pad1): track 0.00 -> 21.8 mm
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
Commit message: Finish routing pcb
Parts:
- added J3: +25, Connector_PinHeader_2.54mm:PinHeader_1x02_P2.54mm_Vertical, F.Cu at (168.9, 85.1)
- added J4: -25, Connector_PinHeader_2.54mm:PinHeader_1x02_P2.54mm_Vertical, F.Cu at (168.9, 72.4)
- moved F2 90.6 mm to (165.1, 100.3), turned to 180 degrees
- moved F1 80.2 mm to (165.1, 61.0), turned to 180 degrees
- moved C12 9.25 mm to (154.9, 87.6)
- moved R22 9.25 mm to (151.1, 82.5)
- moved J2 9.25 mm to (162.6, 72.4)
- moved R21 9.25 mm to (156.2, 72.4)
- moved LS1 9.25 mm to (162.6, 82.5)
- moved Q10 2.84 mm to (144.8, 83.8), turned to 0 degrees
- moved Q9 1.80 mm to (144.8, 74.9), turned to 180 degrees
- moved C3 1.27 mm to (33.0, 86.4)
- moved R5 1.27 mm to (34.3, 62.2)
Connections:
- F1 pad 1: (no net) -> -25V
- F2 pad 1: (no net) -> +25V
Routing:
- net GND: track 0.00 -> 70.5 mm
- net Net-(Q10-Pad1): track 0.00 -> 64.4 mm
- net Net-(C11-Pad1): track 33.9 -> 80.7 mm
- net Net-(D3-Pad1): track 38.8 -> 61.3 mm
- net Net-(Q5-Pad2): track 66.4 -> 87.7 mm
- net Net-(D2-Pad1): track 30.1 -> 49.0 mm
- net Net-(D4-Pad2): track 79.5 -> 97.9 mm
- net +25V: track 0.00 -> 17.9 mm
- net Net-(Q7-Pad2): track 6.66 -> 23.2 mm
- net -25V: track 0.00 -> 14.5 mm
- net Net-(Q9-Pad2): track 0.00 -> 8.89 mm
- net Net-(C8-Pad2): track 18.8 -> 25.9 mm
- net Net-(J1-Pad3): track 0.00 -> 6.35 mm
- net Net-(D2-Pad2): track 38.8 -> 43.2 mm
- net Net-(C10-Pad1): track 71.2 -> 67.4 mm
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Other:
- net class Neutral added: clearance 0.2, trace_width 0.8, via_dia 0.8, via_drill 0.4
