File: stereophonic-amp.sch (KiCad schematic (older format))
At the start: 58 parts, among them J1 DIN-3, J2 Headphones, Q1 ГТ308В, Q10 П217Б, Q2 МП26, Q3 МП26, Q4 МП38А, Q5 МП41А, Q6 МП41А, Q7 ГТ402В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

Commit message: Trace first cascades of amplifier
Parts:
- Q10, Q6, Q9: footprint Connector_PinHeader_1.00mm:PinHeader_1x03_P1.00mm_Vertical -> Connector_PinHeader_2.54mm:PinHeader_1x03_P2.54mm_Vertical
- RV4, RV5: footprint Potentiometer_THT:Potentiometer_Piher_PT-15-V15_Vertical -> Potentiometer_THT:Potentiometer_Piher_PT-10-V10_Vertical
Changed lines of the file:
@@
 F 0 "RV4" V 7243 3400 50  0000 C CNN
 F 1 "1K" V 7334 3400 50  0000 C CNN
-F 2 "Potentiometer_THT:Potentiometer_Piher_PT-15-V15_Vertical" H 7450 3400 50  0001 C CNN
+F 2 "Potentiometer_THT:Potentiometer_Piher_PT-10-V10_Vertical" H 7450 3400 50  0001 C CNN
 F 3 "~" H 7450 3400 50  0001 C CNN
 	1    7450 3400
@@
 F 0 "Q6" H 9790 4396 50  0000 L CNN
 F 1 "МП41А" H 9790 4305 50  0000 L CNN
-F 2 "Connector_PinHeader_1.00mm:PinHeader_1x03_P1.00mm_Vertical" H 9800 4450 50  0001 C CNN
+F 2 "Connector_PinHeader_2.54mm:PinHeader_1x03_P2.54mm_Vertical" H 9800 4450 50  0001 C CNN
 F 3 "~" H 9600 4350 50  0001 C CNN
 	1    9600 4350
@@
 F 0 "RV5" H 9031 2896 50  0000 R CNN
 F 1 "19K" H 9031 2805 50  0000 R CNN
-F 2 "Potentiometer_THT:Potentiometer_Piher_PT-15-V15_Vertical" H 9100 2850 50  0001 C CNN
+F 2 "Potentiometer_THT:Potentiometer_Piher_PT-10-V10_Vertical" H 9100 2850 50  0001 C CNN
 F 3 "~" H 9100 2850 50  0001 C CNN
 	1    9100 2850
@@
 F 0 "Q9" H 11391 2396 50  0000 L CNN
 F 1 "П217Б" H 11391 2305 50  0000 L CNN
-F 2 "Connector_PinHeader_1.00mm:PinHeader_1x03_P1.00mm_Vertical" H 11400 2450 50  0001 C CNN
+F 2 "Connector_PinHeader_2.54mm:PinHeader_1x03_P2.54mm_Vertical" H 11400 2450 50  0001 C CNN
 F 3 "~" H 11200 2350 50  0001 C CNN
 	1    11200 2350
@@
 F 0 "Q10" H 11391 3696 50  0000 L CNN
 F 1 "П217Б" H 11391 3605 50  0000 L CNN
-F 2 "Connector_PinHeader_1.00mm:PinHeader_1x03_P1.00mm_Vertical" H 11400 3750 50  0001 C CNN
+F 2 "Connector_PinHeader_2.54mm:PinHeader_1x03_P2.54mm_Vertical" H 11400 3750 50  0001 C CNN
 F 3 "~" H 11200 3650 50  0001 C CNN
 	1    11200 3650

Commit message: Finish routing pcb
Parts:
- added J3: +25, Connector_PinHeader_2.54mm:PinHeader_1x02_P2.54mm_Vertical, symbol Connector_Generic:Conn_01x02
- added J4: -25, Connector_PinHeader_2.54mm:PinHeader_1x02_P2.54mm_Vertical, symbol Connector_Generic:Conn_01x02
Connections:
- net +25V: now also J3.1 (Pin_1)
- net -25V: now also J4.1 (Pin_1)
- net GND: now also J3.2 (Pin_2), J4.2 (Pin_2)
Changed lines of the file:
@@
 	800  3200 700  3200
 NoConn ~ 700  3200
+$Comp
+L Connector_Generic:Conn_01x02 J3
+U 1 1 60B8690C
+P 15250 1100
+F 0 "J3" H 15330 1092 50  0000 L CNN
+F 1 "+25" H 15330 1001 50  0000 L CNN
+F 2 "Connector_PinHeader_2.54mm:PinHeader_1x02_P2.54mm_Vertical" H 15250 1100 50  0001 C CNN
+F 3 "~" H 15250 1100 50  0001 C CNN
+	1    15250 1100
+	1    0    0    -1
+$EndComp
+$Comp
+L local:+25V #PWR0111
+U 1 1 60B86F30
+P 14850 1100
+F 0 "#PWR0111" H 14850 950 50  0001 C CNN
+F 1 "+25V" H 14865 1273 50  0000 C CNN
+F 2 "" H 14850 1100 50  0001 C CNN
+F 3 "" H 14850 1100 50  0001 C CNN
+	1    14850 1100
+	1    0    0    -1
+$EndComp
+Wire Wire Line
+	15050 1100 14850 1100
+$Comp
+L power:GND #PWR0112
+U 1 1 60B8E2FE
+P 14850 1250
+F 0 "#PWR0112" H 14850 1000 50  0001 C CNN
+F 1 "GND" H 14855 1077 50  0000 C CNN
+F 2 "" H 14850 1250 50  0001 C CNN
+F 3 "" H 14850 1250 50  0001 C CNN
+	1    14850 1250
+	1    0    0    -1
+$EndComp
+Wire Wire Line
+	15050 1200 14850 1200
+Wire Wire Line
+	14850 1200 14850 1250
+$Comp
+L Connector_Generic:Conn_01x02 J4
+U 1 1 60B9BF36
+P 15250 1800
+F 0 "J4" H 15330 1792 50  0000 L CNN
+F 1 "-25" H 15330 1701 50  0000 L CNN
+F 2 "Connector_PinHeader_2.54mm:PinHeader_1x02_P2.54mm_Vertical" H 15250 1800 50  0001 C CNN
+F 3 "~" H 15250 1800 50  0001 C CNN
+	1    15250 1800
+	1    0    0    -1
+$EndComp
+$Comp
+L local:-25V #PWR0113
+U 1 1 60B9C5D8
+P 14850 1750
+F 0 "#PWR0113" H 14850 1600 50  0001 C CNN
+F 1 "-25V" H 14865 1923 50  0000 C CNN
+F 2 "" H 14850 1750 50  0001 C CNN
+F 3 "" H 14850 1750 50  0001 C CNN
+	1    14850 1750
+	1    0    0    -1
+$EndComp
+Wire Wire Line
+	15050 1800 14850 1800
+Wire Wire Line
+	14850 1800 14850 1750
+$Comp
+L power:GND #PWR0114
+U 1 1 60BA3D1A
+P 14850 1950
+F 0 "#PWR0114" H 14850 1700 50  0001 C CNN
+F 1 "GND" H 14855 1777 50  0000 C CNN
+F 2 "" H 14850 1950 50  0001 C CNN
+F 3 "" H 14850 1950 50  0001 C CNN
+	1    14850 1950
+	1    0    0    -1
+$EndComp
+Wire Wire Line
+	15050 1900 14850 1900
+Wire Wire Line
+	14850 1900 14850 1950
 $EndSCHEMATC
